Commit message: fix

File: resources/robots/bennett/bennett.urdf (robot description, URDF)
Before this commit: robot bennett, 17 links, 16 joints
Links:
- link FL-leg-link11: geometry visual mesh filename=meshes/FL-leg-link11.stl
- link FR-leg-link11: geometry visual mesh filename=meshes/FR-leg-link11.stl
- link RL-leg-link11: geometry visual mesh filename=meshes/RL-leg-link11.stl
- link RR-leg-link11: geometry visual mesh filename=meshes/RR-leg-link11.stl
Joints:
- joint FL-Double-Motor1_FL-Motor-Link1_joint: limit lower=-1.570795 upper=1.570795 effort=12 velocity=50 -> lower=-1.570795 upper=1.570795 effort=12 velocity=5
- joint FL-Single-Motor1_FL-Revolute_joint: limit lower=-1.570795 upper=1.570795 effort=12 velocity=50 -> lower=-1.570795 upper=1.570795 effort=12 velocity=5
- joint FL-leg-link11_FL-Link1-Link2_joint: limit lower=-1.570795 upper=1.570795 effort=12 velocity=50 -> lower=-1.570795 upper=1.570795 effort=12 velocity=5
- joint FR-Double-Motor1_FR-Motor-Link1_joint: limit lower=-1.570795 upper=1.570795 effort=12 velocity=50 -> lower=-1.570795 upper=1.570795 effort=12 velocity=5
- joint FR-Single-Motor1_FR-Revolute_joint: limit lower=-1.570795 upper=1.570795 effort=12 velocity=50 -> lower=-1.570795 upper=1.570795 effort=12 velocity=5
- joint FR-leg-link11_FR-Link1-Link2_joint: limit lower=-1.570795 upper=1.570795 effort=12 velocity=50 -> lower=-1.570795 upper=1.570795 effort=12 velocity=5
- joint RL-Double-Motor1_RL-Motor-Link1_joint: limit lower=-1.570795 upper=1.570795 effort=12 velocity=50 -> lower=-1.570795 upper=1.570795 effort=12 velocity=5
- joint RL-Single-Motor1_RL-Revolute_joint: limit lower=-1.570795 upper=1.570795 effort=12 velocity=50 -> lower=-1.570795 upper=1.570795 effort=12 velocity=5
- joint RL-leg-link11_RL-Link1-Link2_joint: limit lower=-1.570795 upper=1.570795 effort=12 velocity=50 -> lower=-1.570795 upper=1.570795 effort=12 velocity=5
- joint RR-Double-Motor1_RR-Motor-Link1_joint: limit lower=-1.570795 upper=1.570795 effort=12 velocity=50 -> lower=-1.570795 upper=1.570795 effort=12 velocity=5
- joint RR-Single-Motor1_RR-Revolute_joint: limit lower=-1.570795 upper=1.570795 effort=12 velocity=50 -> lower=-1.570795 upper=1.570795 effort=12 velocity=5
- joint RR-leg-link11_RR-Link1-Link2_joint: limit lower=-1.570795 upper=1.570795 effort=12 velocity=50 -> lower=-1.570795 upper=1.570795 effort=12 velocity=5

Commit message: better trot modified limit in link11-21 joint:(-1.2 0.4) modified initial pos

File: resources/robots/bennett/bennett.urdf (robot description, URDF)
Before this commit: robot bennett, 17 links, 16 joints
Joints:
- joint FL-Double-Motor1_FL-Motor-Link1_joint: limit lower=-1.570795 upper=1.570795 effort=12 velocity=5 -> lower=-1.570795 upper=1.570795 effort=20 velocity=50
- joint FL-Single-Motor1_FL-Revolute_joint: limit lower=-1.570795 upper=1.570795 effort=12 velocity=5 -> lower=-1.570795 upper=1.570795 effort=20 velocity=50
- joint FL-leg-link11_FL-Link1-Link2_joint: limit lower=-1.570795 upper=1.570795 effort=12 velocity=5 -> lower=-1.2 upper=0.4 effort=20 velocity=50
- joint FR-Double-Motor1_FR-Motor-Link1_joint: limit lower=-1.570795 upper=1.570795 effort=12 velocity=5 -> lower=-1.570795 upper=1.570795 effort=20 velocity=50
- joint FR-Single-Motor1_FR-Revolute_joint: limit lower=-1.570795 upper=1.570795 effort=12 velocity=5 -> lower=-1.570795 upper=1.570795 effort=20 velocity=50
- joint FR-leg-link11_FR-Link1-Link2_joint: limit lower=-1.570795 upper=1.570795 effort=12 velocity=5 -> lower=-1.2 upper=0.4 effort=20 velocity=50
- joint RL-Double-Motor1_RL-Motor-Link1_joint: limit lower=-1.570795 upper=1.570795 effort=12 velocity=5 -> lower=-1.570795 upper=1.570795 effort=20 velocity=50
- joint RL-Single-Motor1_RL-Revolute_joint: limit lower=-1.570795 upper=1.570795 effort=12 velocity=5 -> lower=-1.570795 upper=1.570795 effort=20 velocity=50
- joint RL-leg-link11_RL-Link1-Link2_joint: limit lower=-1.570795 upper=1.570795 effort=12 velocity=5 -> lower=-1.2 upper=0.4 effort=20 velocity=50
- joint RR-Double-Motor1_RR-Motor-Link1_joint: limit lower=-1.570795 upper=1.570795 effort=12 velocity=5 -> lower=-1.570795 upper=1.570795 effort=20 velocity=50
- joint RR-Single-Motor1_RR-Revolute_joint: limit lower=-1.570795 upper=1.570795 effort=12 velocity=5 -> lower=-1.570795 upper=1.570795 effort=20 velocity=50
- joint RR-leg-link11_RR-Link1-Link2_joint: limit lower=-1.570795 upper=1.570795 effort=12 velocity=5 -> lower=-1.2 upper=0.4 effort=20 velocity=50

Commit message: new rl result in Dec22_13_1

File: resources/robots/bennett/bennett.urdf (robot description, URDF)
Before this commit: robot bennett, 17 links, 16 joints
Joints:
- joint FL-Double-Motor1_FL-Motor-Link1_joint: type continuous -> revolute
- joint FL-Single-Motor1_FL-Revolute_joint: type continuous -> revolute
- joint FL-leg-link11_FL-Link1-Link2_joint: type continuous -> revolute
- joint FR-Double-Motor1_FR-Motor-Link1_joint: type continuous -> revolute
- joint FR-Single-Motor1_FR-Revolute_joint: type continuous -> revolute
- joint FR-leg-link11_FR-Link1-Link2_joint: type continuous -> revolute
- joint RL-Double-Motor1_RL-Motor-Link1_joint: type continuous -> revolute
- joint RL-Single-Motor1_RL-Revolute_joint: type continuous -> revolute
- joint RL-leg-link11_RL-Link1-Link2_joint: type continuous -> revolute
- joint RR-Double-Motor1_RR-Motor-Link1_joint: type continuous -> revolute
- joint RR-Single-Motor1_RR-Revolute_joint: type continuous -> revolute
- joint RR-leg-link11_RR-Link1-Link2_joint: type continuous -> revolute
