Commit message: add bennett wheel add bennett real

File: resources/robots/bennett_real/bennett_real.urdf (robot description, URDF)
Before this commit: robot bennett, 17 links, 16 joints
Links:
- link Basic_Body: mass 3.578209936079509 -> 0.5223502772293394
- link FL-Double-Motor1: mass 2.4365544485369104 -> 0.4782524941626558
- link FL-Single-Motor1: mass 0.7011939191100404 -> 0.18505114928963637
- link FL-leg-link11: mass 0.2812248770831842 -> 0.04770813454279477
- link FL-leg-link21: mass 0.2812427717615869 -> 0.03786194092058064
- link FR-Double-Motor1: mass 2.4365544485369104 -> 0.4782524941626558
- link FR-Single-Motor1: mass 0.7011939191100404 -> 0.18505114928963637; geometry collision mesh filename=meshes/FR-Single-Motor1.stl; visual mesh filename=meshes/FR-Single-Motor1.stl
- link FR-leg-link11: mass 0.28122487708301536 -> 0.047708134542766116
- link FR-leg-link21: mass 0.2812427717616486 -> 0.03786194092058894
- link RL-Double-Motor1: mass 2.4365544485369104 -> 0.4782524941626558
- link RL-Single-Motor1: mass 0.7011939191100404 -> 0.18505114928963637; geometry collision mesh filename=meshes/RL-Single-Motor1.stl; visual mesh filename=meshes/RL-Single-Motor1.stl
- link RL-leg-link11: mass 0.2812248770831842 -> 0.04770813454279477
- link RL-leg-link21: mass 0.2812427717615869 -> 0.03786194092058064
- link RR-Double-Motor1: mass 2.4365544485369104 -> 0.4782524941626558
- link RR-Single-Motor1: mass 0.7011939191100404 -> 0.18505114928963637; geometry collision mesh filename=meshes/RR-Single-Motor1.stl; visual mesh filename=meshes/RR-Single-Motor1.stl
- link RR-leg-link11: mass 0.28122487708301536 -> 0.047708134542766116
- link RR-leg-link21: mass 0.2812427717616486 -> 0.03786194092058894
Joints:
- joint FL-Double-Motor1_FL-Motor-Link1_joint: limit lower=-1.570795 upper=1.570795 effort=20 velocity=50 -> lower=-1.570795 upper=1.570795 effort=5 velocity=3.25
- joint FL-Single-Motor1_FL-Revolute_joint: limit lower=-1.570795 upper=1.570795 effort=20 velocity=50 -> lower=-1.570795 upper=1.570795 effort=5 velocity=3.25
- joint FL-leg-link11_FL-Link1-Link2_joint: limit lower=-1.2 upper=0.4 effort=20 velocity=50 -> lower=-1.2 upper=0.4 effort=5 velocity=3.25
- joint FR-Double-Motor1_FR-Motor-Link1_joint: limit lower=-1.570795 upper=1.570795 effort=20 velocity=50 -> lower=-1.570795 upper=1.570795 effort=5 velocity=3.25
- joint FR-Single-Motor1_FR-Revolute_joint: limit lower=-1.570795 upper=1.570795 effort=20 velocity=50 -> lower=-1.570795 upper=1.570795 effort=5 velocity=3.25
- joint FR-leg-link11_FR-Link1-Link2_joint: limit lower=-1.2 upper=0.4 effort=20 velocity=50 -> lower=-1.2 upper=0.4 effort=5 velocity=3.25
- joint RL-Double-Motor1_RL-Motor-Link1_joint: limit lower=-1.570795 upper=1.570795 effort=20 velocity=50 -> lower=-1.570795 upper=1.570795 effort=5 velocity=3.25
- joint RL-Single-Motor1_RL-Revolute_joint: limit lower=-1.570795 upper=1.570795 effort=20 velocity=50 -> lower=-1.570795 upper=1.570795 effort=5 velocity=3.25
- joint RL-leg-link11_RL-Link1-Link2_joint: limit lower=-1.2 upper=0.4 effort=20 velocity=50 -> lower=-1.2 upper=0.4 effort=5 velocity=3.25
- joint RR-Double-Motor1_RR-Motor-Link1_joint: limit lower=-1.570795 upper=1.570795 effort=20 velocity=50 -> lower=-1.570795 upper=1.570795 effort=5 velocity=3.25
- joint RR-Single-Motor1_RR-Revolute_joint: limit lower=-1.570795 upper=1.570795 effort=20 velocity=50 -> lower=-1.570795 upper=1.570795 effort=5 velocity=3.25
- joint RR-leg-link11_RR-Link1-Link2_joint: limit lower=-1.2 upper=0.4 effort=20 velocity=50 -> lower=-1.2 upper=0.4 effort=5 velocity=3.25

File: resources/robots/bennett_wheel/bennett_wheel.urdf (robot description, URDF)
Before this commit: robot bennett_wheel, 25 links, 24 joints
Joints:
- joint FL-leg-link21_FL-leg-link21_FL-Leg-Wheel: limit (none) -> lower=-1.570795 upper=1.570795 effort=20 velocity=50
- joint FR-leg-link21_FR-leg-link21_FR-Leg-Wheel: limit (none) -> lower=-1.570795 upper=1.570795 effort=20 velocity=50
- joint RL-leg-link21_RL-leg-link21_RL-Leg-Wheel: limit (none) -> lower=-1.570795 upper=1.570795 effort=20 velocity=50
- joint RR-leg-link21_RR-leg-link21_RR-Leg-Wheel: limit (none) -> lower=-1.570795 upper=1.570795 effort=20 velocity=50
