Commit message: modified bennett_wheel 1. modified the collision of link21 2. modified the joint limit of link21-link11 3. modified the friction of wheel joint

File: resources/robots/bennett_wheel/bennett_wheel.urdf (robot description, URDF)
Before this commit: robot bennett_wheel, 25 links, 24 joints
Links:
- link FL-leg-link21: geometry collision mesh filename=meshes/FL-leg-link21.stl scale=0.5 0.5 0.5; visual mesh filename=meshes/FL-leg-link21.stl
- link FR-leg-link21: geometry collision mesh filename=meshes/FR-leg-link21.stl scale=0.5 0.5 0.5; visual mesh filename=meshes/FR-leg-link21.stl
- link RL-leg-link21: geometry collision mesh filename=meshes/RL-leg-link21.stl scale=0.5 0.5 0.5; visual mesh filename=meshes/RL-leg-link21.stl
- link RR-leg-link21: geometry collision mesh filename=meshes/RR-leg-link21.stl scale=0.5 0.5 0.5; visual mesh filename=meshes/RR-leg-link21.stl
Joints:
- joint Basic_Body_FL-Body-Single_Motor: limit lower=-1.570795 upper=1.570795 effort=20 velocity=50 -> lower=-1.570795 upper=1.570795 effort=5 velocity=3.25
- joint FL-Double-Motor1_FL-Double_Motor-Link1: limit lower=-1.570795 upper=1.570795 effort=20 velocity=50 -> lower=-1.570795 upper=1.570795 effort=5 velocity=3.25
- joint FL-Single-Motor1_FL-Single-Double_Motor: limit lower=-1.570795 upper=1.570795 effort=20 velocity=50 -> lower=-1.570795 upper=1.570795 effort=5 velocity=3.25
- joint FL-leg-link11_FL-Link1-Link2: limit lower=-1.570795 upper=1.570795 effort=20 velocity=50 -> lower=-1.2 upper=0.4 effort=5 velocity=3.25
- joint FL-leg-link21_FL-leg-link21_FL-Leg-Wheel: limit lower=-1.570795 upper=1.570795 effort=20 velocity=50 -> lower=-1000 upper=1000 effort=10 velocity=50
- joint FR-Double-Motor1_FR-Double_Motor-Link1: limit lower=-1.570795 upper=1.570795 effort=20 velocity=50 -> lower=-1.570795 upper=1.570795 effort=5 velocity=3.25
- joint FR-Single-Motor1_FR-Single-Double_Motor: limit lower=-1.570795 upper=1.570795 effort=20 velocity=50 -> lower=-1.570795 upper=1.570795 effort=5 velocity=3.25
- joint FR-leg-link11_FR-Link1-Link2: limit lower=-1.570795 upper=1.570795 effort=20 velocity=50 -> lower=-1.2 upper=0.4 effort=5 velocity=3.25
- joint FR-leg-link21_FR-leg-link21_FR-Leg-Wheel: limit lower=-1.570795 upper=1.570795 effort=20 velocity=50 -> lower=-1000 upper=1000 effort=5 velocity=50
- joint RL-Double-Motor1_RL-Double_Motor-Link1: limit lower=-1.570795 upper=1.570795 effort=20 velocity=50 -> lower=-1.570795 upper=1.570795 effort=5 velocity=3.25
- joint RL-Single-Motor1_RL-Single-Double_Motor: limit lower=-1.570795 upper=1.570795 effort=20 velocity=50 -> lower=-1.570795 upper=1.570795 effort=5 velocity=3.25
- joint RL-leg-link11_RL-Link1-Link2: limit lower=-1.570795 upper=1.570795 effort=20 velocity=50 -> lower=-1.2 upper=0.4 effort=5 velocity=3.25
- joint RL-leg-link21_RL-leg-link21_RL-Leg-Wheel: limit lower=-1.570795 upper=1.570795 effort=20 velocity=50 -> lower=-1000 upper=1000 effort=10 velocity=50
- joint RR-Double-Motor1_RR-Double_Motor-Link1: limit lower=-1.570795 upper=1.570795 effort=20 velocity=50 -> lower=-1.570795 upper=1.570795 effort=5 velocity=3.25
- joint RR-Single-Motor1_RR-Single-Double_Motor: limit lower=-1.570795 upper=1.570795 effort=20 velocity=50 -> lower=-1.570795 upper=1.570795 effort=5 velocity=3.25
- joint RR-leg-link11_RR-Link1-Link2: limit lower=-1.570795 upper=1.570795 effort=20 velocity=50 -> lower=-1.2 upper=0.4 effort=5 velocity=3.25
- joint RR-leg-link21_RR-Link2-Fingertip: limit lower=-1.570795 upper=1.570795 effort=20 velocity=50 -> (none)
- joint RR-leg-link21_RR-leg-link21_RR-Leg-Wheel: limit lower=-1.570795 upper=1.570795 effort=20 velocity=50 -> lower=-1000 upper=1000 effort=5 velocity=50
