Commit message: wheel

File: resources/robots/bennett_foot/bennett_foot.urdf (robot description, URDF)
Before this commit: robot bennett_foot, 21 links, 20 joints
Links:
- removed link Basic_Body
- added link Body1, mass 3.578209936079509; collision mesh filename=meshes/Body1.stl; visual mesh filename=meshes/Body1.stl
- added link FL-leg-link31, mass 0.24917982527134377; collision mesh filename=meshes/FL-leg-link31.stl; visual mesh filename=meshes/FL-leg-link31.stl
- added link FL-leg-link41, mass 0.30627894117127225; collision mesh filename=meshes/FL-leg-link41.stl; visual mesh filename=meshes/FL-leg-link41.stl
- added link FR-leg-link31, mass 0.24917982527179094; collision mesh filename=meshes/FR-leg-link31.stl; visual mesh filename=meshes/FR-leg-link31.stl
- added link FR-leg-link41, mass 0.30627948094211754; collision mesh filename=meshes/FR-leg-link41.stl; visual mesh filename=meshes/FR-leg-link41.stl
- added link RL-leg-link31, mass 0.24917982527134377; collision mesh filename=meshes/RL-leg-link31.stl; visual mesh filename=meshes/RL-leg-link31.stl
- added link RL-leg-link41, mass 0.30627894117127225; collision mesh filename=meshes/RL-leg-link41.stl; visual mesh filename=meshes/RL-leg-link41.stl
- added link RR-leg-link31, mass 0.24917982527179094; collision mesh filename=meshes/RR-leg-link31.stl; visual mesh filename=meshes/RR-leg-link31.stl
- added link RR-leg-link41, mass 0.30627948094211754; collision mesh filename=meshes/RR-leg-link41.stl; visual mesh filename=meshes/RR-leg-link41.stl
- link FL-Double-Motor1: geometry collision mesh filename=meshes/FL-Double-Motor1.stl; visual mesh filename=meshes/FL-Double-Motor1.stl
- link FL-Single-Motor1: geometry collision mesh filename=meshes/FL-Single-Motor1.stl; visual mesh filename=meshes/FL-Single-Motor1.stl
- link FL-leg-link11: geometry collision mesh filename=meshes/FL-leg-link11.stl; visual mesh filename=meshes/FL-leg-link11.stl
- link FR-Double-Motor1: geometry collision mesh filename=meshes/FR-Double-Motor1.stl; visual mesh filename=meshes/FR-Double-Motor1.stl
- link FR-Single-Motor1: geometry collision mesh filename=meshes/FR-Single-Motor1.stl; visual mesh filename=meshes/FR-Single-Motor1.stl
- link FR-leg-link11: mass 0.2812248770831842 -> 0.28122487708301536; geometry collision mesh filename=meshes/FR-leg-link11.stl; visual mesh filename=meshes/FR-leg-link11.stl
- link FR-leg-link21: mass 0.27918764656736367 -> 0.2791876465674252
- link RL-Double-Motor1: geometry collision mesh filename=meshes/RL-Double-Motor1.stl; visual mesh filename=meshes/RL-Double-Motor1.stl
- link RL-Single-Motor1: geometry collision mesh filename=meshes/RL-Single-Motor1.stl; visual mesh filename=meshes/RL-Single-Motor1.stl
- link RL-leg-link11: geometry collision mesh filename=meshes/RL-leg-link11.stl; visual mesh filename=meshes/RL-leg-link11.stl
- link RR-Double-Motor1: geometry collision mesh filename=meshes/RR-Double-Motor1.stl; visual mesh filename=meshes/RR-Double-Motor1.stl
- link RR-Single-Motor1: geometry collision mesh filename=meshes/RR-Single-Motor1.stl; visual mesh filename=meshes/RR-Single-Motor1.stl
- link RR-leg-link11: mass 0.2812248770831842 -> 0.28122487708301536; geometry collision mesh filename=meshes/RR-leg-link11.stl; visual mesh filename=meshes/RR-leg-link11.stl
- link RR-leg-link21: mass 0.27918764656736367 -> 0.2791876465674252
Joints:
- added joint FL-Double-Motor1_FL-Double_Motor-Link4: type continuous, parent FL-Double-Motor1, child FL-leg-link41, origin xyz=-0.08224999999999998 0.041000000000000016 0.07101407999999998 rpy=-1.5707963267948968 -3.8518598887744726e-34 4.810976478165954e-50, axis 0.0 -0.866025 0.5
- added joint FL-leg-link21_FL-Link2-Link3: type continuous, parent FL-leg-link21, child FL-leg-link31, origin xyz=0.045870350000000004 0.10436275957666326 -0.07044621311142345 rpy=-2.1862760354652835 -0.523598775598294 2.5261129449194093, axis -0.6711405018682711 0.20534699999999997 0.712322400804583
- added joint FL-leg-link41_FL-Link4-Link3: type continuous, parent FL-leg-link41, child FL-leg-link31, origin xyz=0.04450177 -0.05645856000000002 -0.11336067 rpy=-0.7853981633974534 -4.1053665947016125e-48 -1.1102230246251565e-16, axis 0.6644629999999999 0.6204190253469806 0.4166167088733992
- added joint FR-Double-Motor1_FR-Double_Motor-Link4: type continuous, parent FR-Double-Motor1, child FR-leg-link41, origin xyz=-0.08225 0.041000000000000016 -0.07101408 rpy=-1.5707963267948968 -1.5407439555097887e-33 1.9243905912663812e-49, axis 0.0 0.866025 0.5
- added joint FR-leg-link21_FR-Link2-Link3: type continuous, parent FR-leg-link21, child FR-leg-link31, origin xyz=0.045870350000000004 -0.10436275957666319 -0.07044621311142345 rpy=-0.9553166181245096 -0.5235987755982938 -2.5261129449194093, axis 0.671140501868271 -0.20534699999999997 0.7123224008045831
- added joint FR-leg-link41_FR-Link4-Link3: type continuous, parent FR-leg-link41, child FR-leg-link31, origin xyz=0.04450177 0.05645856000000002 -0.11336067 rpy=-2.35619449019234 2.775557561562892e-17 0.0, axis 0.6644629999999999 0.6204190253469807 -0.4166167088733998
- added joint RL-Double-Motor1_RL-Double_Motor-Link4: type continuous, parent RL-Double-Motor1, child RL-leg-link41, origin xyz=0.08225 0.041000000000000016 0.07101408 rpy=-1.5707963267948968 -9.860761315262648e-32 1.7789921910373654e-47, axis 8.539665818050335e-32 -0.866025 0.5
- added joint RL-leg-link21_RL-Link2-Link3: type continuous, parent RL-leg-link21, child RL-leg-link31, origin xyz=0.053980549999999974 0.10323441514378821 -0.06623518009742323 rpy=-2.1862760354652835 -0.523598775598294 2.5261129449194093, axis -0.7123224008045759 0.20534699999999995 0.6711405018682787
- added joint RL-leg-link41_RL-Link4-Link3: type continuous, parent RL-leg-link41, child RL-leg-link31, origin xyz=0.055349129999999996 -0.054278770000000025 -0.10958516000000003 rpy=2.35619449019234 1.1102230246251565e-16 -1.1102230246251556e-16, axis -0.6408559999999999 0.6056687778914289 0.47166638600233346
- added joint RR-Double-Motor1_RR-Double_Motor-Link4: type continuous, parent RR-Double-Motor1, child RR-leg-link41, origin xyz=0.08225 0.041000000000000016 -0.07101407999999998 rpy=-1.5707963267948968 6.162975822039155e-33 -7.697562365065525e-49, axis 0.0 0.8660250000000003 0.5000000000000001
- added joint RR-leg-link21_RR-Link2-Link3: type continuous, parent RR-leg-link21, child RR-leg-link31, origin xyz=0.053980549999999995 -0.10323441514378821 -0.06623518009742321 rpy=-0.9553166181245095 -0.523598775598294 -2.5261129449194097, axis 0.712322400804576 -0.205347 0.6711405018682788
- added joint RR-leg-link41_RR-Link4-Link3: type continuous, parent RR-leg-link41, child RR-leg-link31, origin xyz=0.055349129999999996 0.054278770000000025 -0.10958516000000003 rpy=-2.35619449019234 5.551115123125784e-17 -5.551115123125784e-17, axis 0.6408559999999999 0.6056687778914288 -0.4716663860023348
- joint Body1_FL-Body-Single_Motor: parent Basic_Body -> Body1
- joint Body1_FR-Body-Single_Motor: parent Basic_Body -> Body1
- joint Body1_RL-Body-Single_Motor: parent Basic_Body -> Body1
- joint Body1_RR-Body-Single_Motor: parent Basic_Body -> Body1
- joint FL-Double-Motor1_FL-Double_Motor-Link1: type revolute -> continuous
- joint FL-Single-Motor1_FL-Single-Double_Motor: type revolute -> continuous
- joint FL-leg-link11_FL-Link1-Link2: axis 0.619449 -0.5947552918305997 -0.5123957365986744 -> 0.640856 -0.6056687778914328 -0.47166638600232924; origin xyz=-0.06338258 -0.06892026 -0.09654496000000001 rpy=-0.7853981633974451 5.551115123125784e-17 -5.551115123125782e-17 -> xyz=-0.055349129999999996 -0.07090645000000001 -0.09998516000000002 rpy=-0.7853981633974451 5.551115123125783e-17 6.798155367234457e-33; type revolute -> continuous
- joint FL-leg-link21_FL-Link2-Fingertip: origin xyz=0.08605386 0.13816643058642264 -0.052438275217471075 rpy=-2.356194490192348 -2.453269466693416e-17 -5.397192826725469e-17 -> xyz=0.05896426999999999 0.1342397322802053 -0.08802220068595261 rpy=-2.356194490192348 -2.453269466693391e-17 2.453269466693407e-17
- joint FR-Double-Motor1_FR-Double_Motor-Link1: axis -5.293503193065871e-33 0.8589199999999999 0.5121090000000001 -> 0.0 0.8660249999999999 0.5000000000000001; origin xyz=-0.08225 0.03216045999999999 -0.053940199999999994 rpy=-1.5707963267948968 -7.703719777548943e-33 9.621952956331906e-49 -> xyz=-0.08225 0.031400000000000004 -0.054386399999999994 rpy=-1.5707963267948968 -1.5407439555097887e-33 1.9243905912663812e-49; type revolute -> continuous
- joint FR-Single-Motor1_FR-Single-Double_Motor: type revolute -> continuous
- joint FR-leg-link11_FR-Link1-Link2: axis -0.678696 0.365770781558617 0.6368543082621005 -> -0.640856 -0.6056687778914328 0.47166638600232924; origin xyz=0.0362449 0.07587255000000002 -0.10496640999999997 rpy=-0.7853981633974451 -2.7755575615628914e-17 2.7638981384219264e-33 -> xyz=-0.055349129999999996 0.07090645000000004 -0.09998516000000002 rpy=0.7853981633974454 -0.0 0.0; type revolute -> continuous
- joint FR-leg-link21_FR-Link2-Fingertip: origin xyz=-0.05290837999999999 0.10801814101093907 -0.1215639169175536 rpy=-2.356194490192348 -4.906538933386794e-17 9.813077866773741e-18 -> xyz=0.05896426999999999 -0.13423973228020525 -0.0880222006859526 rpy=2.356194490192348 -5.3971928267254846e-17 2.453269466693382e-17
- joint RL-Double-Motor1_RL-Double_Motor-Link1: type revolute -> continuous
- joint RL-Single-Motor1_RL-Single-Double_Motor: type revolute -> continuous
- joint RL-leg-link11_RL-Link1-Link2: axis 0.659865 -0.6172412874723316 -0.4284748895938925 -> 0.664463 -0.6204190253469839 -0.41661670887339414; origin xyz=-0.04683741999999997 -0.07266289 -0.10302739000000002 rpy=-0.7853981633974451 -1.2075949781892453e-47 9.860761315262648e-32 -> xyz=-0.04450176999999998 -0.07308624 -0.10376067 rpy=-0.7853981633974451 2.7755575615628907e-17 5.551115123125793e-17; type revolute -> continuous
- joint RL-leg-link21_RL-Link2-Fingertip: origin xyz=0.0670498 0.13311853669688808 -0.08383781852653531 rpy=-2.356194490192348 -9.813077866773564e-18 9.813077866773624e-18 -> xyz=0.06917824999999998 0.1327916836583524 -0.08261801690258165 rpy=-2.356194490192348 1.9626155733547254e-17 1.962615573354713e-17
- joint RR-Double-Motor1_RR-Double_Motor-Link1: type revolute -> continuous
- joint RR-Single-Motor1_RR-Single-Double_Motor: type revolute -> continuous
- joint RR-leg-link11_RR-Link1-Link2: axis -0.579228 0.574772454194268 0.5780407017369087 -> -0.664463 -0.620419025346984 0.4166167088733942; origin xyz=0.07570079 0.06517376000000004 -0.09005584999999997 rpy=-0.7853981633974451 -5.551115123125784e-17 5.551115123125782e-17 -> xyz=-0.04450176999999998 0.07308624000000004 -0.10376067 rpy=0.7853981633974454 -6.798155367234455e-33 5.551115123125783e-17; type revolute -> continuous
- joint RR-leg-link21_RR-Link2-Fingertip: origin xyz=-0.03727120999999997 0.09615481962414142 -0.13641886567419534 rpy=-2.3561944901923475 7.459472472164641e-17 8.241452114673111e-17 -> xyz=0.06917825000000001 -0.13279168365835242 -0.08261801690258162 rpy=2.356194490192348 -3.925231146709402e-17 -1.1775693440128322e-16

File: resources/robots/bennett_real/bennett_real.urdf (robot description, URDF)
Before this commit: robot Quadruped-IsaacSim, 17 links, 16 joints
Links:
- removed link Basic_Body
- added link Body1, mass 0.5223502772293394; collision mesh filename=meshes/Body1.stl; visual mesh filename=meshes/Body1.stl
- added link FL-leg-link31, mass 0.030992351814191726; collision mesh filename=meshes/FL-leg-link31.stl; visual mesh filename=meshes/FL-leg-link31.stl
- added link FL-leg-link41, mass 0.049054688661482895; collision mesh filename=meshes/FL-leg-link41.stl; visual mesh filename=meshes/FL-leg-link41.stl
- added link FR-leg-link31, mass 0.030992351814247344; collision mesh filename=meshes/FR-leg-link31.stl; visual mesh filename=meshes/FR-leg-link31.stl
- added link FR-leg-link41, mass 0.04905477511303801; collision mesh filename=meshes/FR-leg-link41.stl; visual mesh filename=meshes/FR-leg-link41.stl
- added link RL-leg-link31, mass 0.030992351814191726; collision mesh filename=meshes/RL-leg-link31.stl; visual mesh filename=meshes/RL-leg-link31.stl
- added link RL-leg-link41, mass 0.049054688661482895; collision mesh filename=meshes/RL-leg-link41.stl; visual mesh filename=meshes/RL-leg-link41.stl
- added link RR-leg-link31, mass 0.030992351814247344; collision mesh filename=meshes/RR-leg-link31.stl; visual mesh filename=meshes/RR-leg-link31.stl
- added link RR-leg-link41, mass 0.04905477511303801; collision mesh filename=meshes/RR-leg-link41.stl; visual mesh filename=meshes/RR-leg-link41.stl
- link FL-Double-Motor1: geometry collision mesh filename=meshes/FL-Double-Motor1.stl; visual mesh filename=meshes/FL-Double-Motor1.stl
- link FL-leg-link11: geometry collision mesh filename=meshes/FL-leg-link11.stl; visual mesh filename=meshes/FL-leg-link11.stl
- link FR-Double-Motor1: geometry collision mesh filename=meshes/FR-Double-Motor1.stl; visual mesh filename=meshes/FR-Double-Motor1.stl
- link FR-leg-link11: geometry collision mesh filename=meshes/FR-leg-link11.stl; visual mesh filename=meshes/FR-leg-link11.stl
- link RL-Double-Motor1: geometry collision mesh filename=meshes/RL-Double-Motor1.stl; visual mesh filename=meshes/RL-Double-Motor1.stl
- link RL-leg-link11: geometry collision mesh filename=meshes/RL-leg-link11.stl; visual mesh filename=meshes/RL-leg-link11.stl
- link RR-Double-Motor1: geometry collision mesh filename=meshes/RR-Double-Motor1.stl; visual mesh filename=meshes/RR-Double-Motor1.stl
- link RR-leg-link11: geometry collision mesh filename=meshes/RR-leg-link11.stl; visual mesh filename=meshes/RR-leg-link11.stl
Joints:
- removed joint Basic_Body_FL-Rigid
- removed joint Basic_Body_FR-Rigid
- removed joint Basic_Body_RL-Rigid
- removed joint Basic_Body_RR-Rigid
- removed joint FL-Double-Motor1_FL-Motor-Link1_joint
- removed joint FL-Single-Motor1_FL-Revolute_joint
- removed joint FL-leg-link11_FL-Link1-Link2_joint
- removed joint FR-Double-Motor1_FR-Motor-Link1_joint
- removed joint FR-Single-Motor1_FR-Revolute_joint
- removed joint FR-leg-link11_FR-Link1-Link2_joint
- removed joint RL-Double-Motor1_RL-Motor-Link1_joint
- removed joint RL-Single-Motor1_RL-Revolute_joint
- removed joint RL-leg-link11_RL-Link1-Link2_joint
- removed joint RR-Double-Motor1_RR-Motor-Link1_joint
- removed joint RR-Single-Motor1_RR-Revolute_joint
- removed joint RR-leg-link11_RR-Link1-Link2_joint
- added joint Body1_FL-Rigid: type fixed, parent Body1, child FL-Single-Motor1, origin xyz=-0.044000000000000004 -0.032 0.012000000000000028 rpy=3.141592653589793 -0.0 0.0
- added joint Body1_FR-Rigid: type fixed, parent Body1, child FR-Single-Motor1, origin xyz=-0.044000000000000004 0.029500000000000002 0.012000000000000028 rpy=3.141592653589793 -0.0 0.0
- added joint Body1_RL-Rigid: type fixed, parent Body1, child RL-Single-Motor1, origin xyz=0.044000000000000004 -0.032 0.012000000000000028 rpy=3.141592653589793 -0.0 0.0
- added joint Body1_RR-Rigid: type fixed, parent Body1, child RR-Single-Motor1, origin xyz=0.044000000000000004 0.029500000000000002 0.012000000000000028 rpy=3.141592653589793 -0.0 0.0
- added joint FL-Double-Motor1_FL-Motor-Link1: type continuous, parent FL-Double-Motor1, child FL-leg-link11, origin xyz=-0.08225 0.031400000000000004 0.054386399999999994 rpy=-1.5707963267948968 1.0785207688568522e-32 5.551115123125783e-17, axis 2.775557561562891e-17 -0.8660250000000002 0.4999999999999999
- added joint FL-Double-Motor1_FL-Motor-Link4: type continuous, parent FL-Double-Motor1, child FL-leg-link41, origin xyz=-0.08225 0.041000000000000016 0.07101408 rpy=-1.5707963267948968 1.0785207688568522e-32 5.551115123125783e-17, axis 2.775557561562891e-17 -0.866025 0.5
- added joint FL-Single-Motor1_FL-Revolute: type continuous, parent FL-Single-Motor1, child FL-Double-Motor1, origin xyz=-0.034499999999999996 0.03925 0.016750000000000043 rpy=-1.5707963267948966 -0.0 0.0, axis -1.0 0.0 7.806255641895643e-18
- added joint FL-leg-link11_FL-Link1-Link2: type continuous, parent FL-leg-link11, child FL-leg-link21, origin xyz=-0.06577526000000003 -0.06826225 -0.09540526999999997 rpy=-0.7853981633974452 5.551115123125784e-17 -5.551115123125784e-17, axis 0.6123719999999999 -0.5915061361710475 -0.5245190823621178
- added joint FL-leg-link21_FL-Link2-Link3: type continuous, parent FL-leg-link21, child FL-leg-link31, origin xyz=0.03741105000000001 0.10530386213388003 -0.07395845491998392 rpy=-2.1862760354652835 -0.5235987755982939 2.5261129449194093, axis -0.6283202365199574 0.20095100000000005 0.7515533921315938
- added joint FL-leg-link41_FL-Link4-Link3: type continuous, parent FL-leg-link41, child FL-leg-link31, origin xyz=0.033315729999999974 -0.05815736000000001 -0.11630306999999998 rpy=-0.7853981633974534 8.326672684688675e-17 -3.851859888774471e-33, axis 0.6830129999999999 0.6356458627730519 0.35978936529656114
- added joint FR-Double-Motor1_FR-Motor-Link1: type continuous, parent FR-Double-Motor1, child FR-leg-link11, origin xyz=-0.08225 0.031400000000000004 -0.054386399999999994 rpy=-1.5707963267948968 -6.93334779979405e-33 -5.551115123125783e-17, axis -2.7755575615628914e-17 0.8660249999999999 0.5000000000000001
- added joint FR-Double-Motor1_FR-Motor-Link4: type continuous, parent FR-Double-Motor1, child FR-leg-link41, origin xyz=-0.08225 0.041000000000000016 -0.07101408 rpy=-1.5707963267948968 -6.93334779979405e-33 -5.551115123125783e-17, axis -2.7755575615628914e-17 0.866025 0.5
- added joint FR-Single-Motor1_FR-Revolute: type continuous, parent FR-Single-Motor1, child FR-Double-Motor1, origin xyz=-0.034499999999999996 -0.03925 0.016750000000000043 rpy=-1.5707963267948966 -0.0 0.0, axis -1.0 -2.465190328815662e-32 7.806255641895643e-18
- added joint FR-leg-link11_FR-Link1-Link2: type continuous, parent FR-leg-link11, child FR-leg-link21, origin xyz=-0.06577526000000003 0.06826225000000002 -0.09540526999999997 rpy=-2.356194490192348 -5.551115123125782e-17 -5.551115123125784e-17, axis 0.612372 -0.5915061361710475 0.5245190823621178
- added joint FR-leg-link21_FR-Link2-Link3: type continuous, parent FR-leg-link21, child FR-leg-link31, origin xyz=0.037411049999999973 0.10530386213387996 0.07395845491998396 rpy=2.1862760354652835 -0.5235987755982939 -2.5261129449194097, axis 0.7515533921315871 0.20095100000000002 -0.6283202365199652
- added joint FR-leg-link41_FR-Link4-Link3: type continuous, parent FR-leg-link41, child FR-leg-link31, origin xyz=0.03331573000000001 0.05815736000000001 -0.11630306999999998 rpy=-2.35619449019234 -5.551115123125783e-17 5.551115123125783e-17, axis 0.683013 0.635645862773052 -0.3597893652965619
- added joint RL-Double-Motor1_RL-Motor-Link1: type continuous, parent RL-Double-Motor1, child RL-leg-link11, origin xyz=0.08225 0.031400000000000004 0.054386399999999994 rpy=-1.5707963267948968 -9.860761315262648e-32 1.2316099784104838e-47, axis 8.539665818050335e-32 -0.8660250000000002 0.4999999999999999
- added joint RL-Double-Motor1_RL-Motor-Link4: type continuous, parent RL-Double-Motor1, child RL-leg-link41, origin xyz=0.08225 0.041000000000000016 0.07101408 rpy=-1.5707963267948968 -9.860761315262648e-32 1.2316099784104838e-47, axis 8.539665818050335e-32 -0.866025 0.5
- added joint RL-Single-Motor1_RL-Revolute: type continuous, parent RL-Single-Motor1, child RL-Double-Motor1, origin xyz=0.034499999999999996 0.03925 0.016750000000000043 rpy=-1.5707963267948966 6.077163357286271e-64 0.0, axis 1.0 4.930380657631324e-32 -7.806255641895643e-18
- added joint RL-leg-link11_RL-Link1-Link2: type continuous, parent RL-leg-link11, child RL-leg-link21, origin xyz=-0.04450177 -0.07308624 -0.10376067 rpy=-0.7853981633974451 6.798155367234458e-33 -5.551115123125773e-17, axis 0.664463 -0.620419025346984 -0.416616708873394
- added joint RL-leg-link21_RL-Link2-Link3: type continuous, parent RL-leg-link21, child RL-leg-link31, origin xyz=0.053980549999999995 0.10323441514378828 -0.06623518009742323 rpy=0.9553166181245096 -0.5235987755982939 2.5261129449194097, axis 0.712322400804576 0.20534700000000003 0.6711405018682788
- added joint RL-leg-link41_RL-Link4-Link3: type continuous, parent RL-leg-link41, child RL-leg-link31, origin xyz=0.055349129999999996 -0.054278770000000025 -0.10958516000000003 rpy=-0.7853981633974534 5.551115123125783e-17 9.860761315262648e-32, axis 0.640856 0.6056687778914289 0.4716663860023341
- added joint RR-Double-Motor1_RR-Motor-Link1: type continuous, parent RR-Double-Motor1, child RR-leg-link11, origin xyz=0.08224999999999998 0.031400000000000004 -0.05438639999999999 rpy=-1.5707963267948968 -4.9303806576313227e-32 6.07716335728627e-64, axis -4.2698329090251674e-32 0.8660249999999999 0.5000000000000002
- added joint RR-Double-Motor1_Revolute_45: type continuous, parent RR-Double-Motor1, child RR-leg-link41, origin xyz=0.08224999999999998 0.041000000000000016 -0.07101407999999998 rpy=-1.5707963267948966 -4.9303806576313227e-32 6.07716335728627e-64, axis -4.2698329090251674e-32 0.866025 0.5000000000000001
- added joint RR-Single-Motor1_RR-Revolute: type continuous, parent RR-Single-Motor1, child RR-Double-Motor1, origin xyz=0.034499999999999996 -0.03925 0.016750000000000043 rpy=-1.5707963267948966 -0.0 0.0, axis 0.9999999999999999 -3.851859888774472e-34 0.0
- added joint RR-leg-link11_RR-Link1-Link2: type continuous, parent RR-leg-link11, child RR-leg-link21, origin xyz=-0.04450177 0.07308624000000004 -0.10376066999999992 rpy=-2.356194490192348 -6.798155367234463e-33 5.551115123125789e-17, axis 0.664463 -0.620419025346984 0.4166167088733941
- added joint RR-leg-link21_Revolute_47: type continuous, parent RR-leg-link21, child RR-leg-link31, origin xyz=0.053980550000000016 0.10323441514378821 0.06623518009742321 rpy=2.1862760354652835 -0.5235987755982938 -2.5261129449194093, axis 0.671140501868271 0.20534699999999995 -0.7123224008045831
- added joint RR-leg-link41_Revolute_46: type continuous, parent RR-leg-link41, child RR-leg-link31, origin xyz=0.055349129999999996 0.054278770000000025 -0.10958515999999996 rpy=-2.35619449019234 -0.0 5.551115123125789e-17, axis 0.640856 0.6056687778914288 -0.4716663860023341

File: resources/robots/bennett_wheel/bennett_wheel.urdf (robot description, URDF)
Before this commit: robot bennett_wheel, 25 links, 24 joints
Joints:
- joint FL-leg-link21_FL-leg-link21_FL-Leg-Wheel: limit lower=-1000 upper=1000 effort=10 velocity=50 -> lower=-1e6 upper=1e6 effort=10 velocity=50; type continuous -> revolute
- joint FR-leg-link21_FR-leg-link21_FR-Leg-Wheel: limit lower=-1000 upper=1000 effort=5 velocity=50 -> lower=-1e6 upper=1e6 effort=5 velocity=50; type continuous -> revolute
- joint RL-leg-link21_RL-leg-link21_RL-Leg-Wheel: limit lower=-1000 upper=1000 effort=10 velocity=50 -> lower=-1e6 upper=1e6 effort=10 velocity=50; type continuous -> revolute
- joint RR-leg-link21_RR-leg-link21_RR-Leg-Wheel: limit lower=-1000 upper=1000 effort=5 velocity=50 -> lower=-1e6 upper=1e6 effort=5 velocity=50; type continuous -> revolute
